File: input_buffer_bal_XLR_combo_SMD_1206.sch (KiCad schematic (older format))
At the start: 31 parts, among them J1 CH1, J2 CH2, J3 POWER, J4 CH1_OUT, J5 CH2_OUT, U1 LM4562, U2 LM4562

Commit message: minor improvements
Parts:
- C1, C2, C3, C4, C5, C6, C7, C8: footprint Capacitor_SMD:C_1206_3216Metric -> Capacitor_SMD:C_1206_3216Metric_Pad1.42x1.75mm_HandSolder
Changed lines of the file:
@@
 F 0 "C5" H 4615 1796 50  0000 L CNN
 F 1 "220p" H 4615 1705 50  0000 L CNN
-F 2 "Capacitor_SMD:C_1206_3216Metric" H 4538 1600 50  0001 C CNN
+F 2 "Capacitor_SMD:C_1206_3216Metric_Pad1.42x1.75mm_HandSolder" H 4538 1600 50  0001 C CNN
 F 3 "~" H 4500 1750 50  0001 C CNN
 	1    4500 1750
@@
 F 0 "C6" H 4615 2296 50  0000 L CNN
 F 1 "220p" H 4615 2205 50  0000 L CNN
-F 2 "Capacitor_SMD:C_1206_3216Metric" H 4538 2100 50  0001 C CNN
+F 2 "Capacitor_SMD:C_1206_3216Metric_Pad1.42x1.75mm_HandSolder" H 4538 2100 50  0001 C CNN
 F 3 "~" H 4500 2250 50  0001 C CNN
 	1    4500 2250
@@
 F 0 "C7" H 4615 3796 50  0000 L CNN
 F 1 "220p" H 4615 3705 50  0000 L CNN
-F 2 "Capacitor_SMD:C_1206_3216Metric" H 4538 3600 50  0001 C CNN
+F 2 "Capacitor_SMD:C_1206_3216Metric_Pad1.42x1.75mm_HandSolder" H 4538 3600 50  0001 C CNN
 F 3 "~" H 4500 3750 50  0001 C CNN
 	1    4500 3750
@@
 F 0 "C8" H 4615 4296 50  0000 L CNN
 F 1 "220p" H 4615 4205 50  0000 L CNN
-F 2 "Capacitor_SMD:C_1206_3216Metric" H 4538 4100 50  0001 C CNN
+F 2 "Capacitor_SMD:C_1206_3216Metric_Pad1.42x1.75mm_HandSolder" H 4538 4100 50  0001 C CNN
 F 3 "~" H 4500 4250 50  0001 C CNN
 	1    4500 4250
@@
 F 0 "C3" H 3565 6296 50  0000 L CNN
 F 1 "100n" H 3565 6205 50  0000 L CNN
-F 2 "Capacitor_SMD:C_1206_3216Metric" H 3488 6100 50  0001 C CNN
+F 2 "Capacitor_SMD:C_1206_3216Metric_Pad1.42x1.75mm_HandSolder" H 3488 6100 50  0001 C CNN
 F 3 "~" H 3450 6250 50  0001 C CNN
 	1    3450 6250
@@
 F 0 "C4" H 4015 6296 50  0000 L CNN
 F 1 "100n" H 4015 6205 50  0000 L CNN
-F 2 "Capacitor_SMD:C_1206_3216Metric" H 3938 6100 50  0001 C CNN
+F 2 "Capacitor_SMD:C_1206_3216Metric_Pad1.42x1.75mm_HandSolder" H 3938 6100 50  0001 C CNN
 F 3 "~" H 3900 6250 50  0001 C CNN
 	1    3900 6250
@@
 F 0 "C1" H 1715 5996 50  0000 L CNN
 F 1 "100n" H 1715 5905 50  0000 L CNN
-F 2 "Capacitor_SMD:C_1206_3216Metric" H 1638 5800 50  0001 C CNN
+F 2 "Capacitor_SMD:C_1206_3216Metric_Pad1.42x1.75mm_HandSolder" H 1638 5800 50  0001 C CNN
 F 3 "~" H 1600 5950 50  0001 C CNN
 	1    1600 5950
@@
 F 0 "C2" H 2165 5996 50  0000 L CNN
 F 1 "100n" H 2165 5905 50  0000 L CNN
-F 2 "Capacitor_SMD:C_1206_3216Metric" H 2088 5800 50  0001 C CNN
+F 2 "Capacitor_SMD:C_1206_3216Metric_Pad1.42x1.75mm_HandSolder" H 2088 5800 50  0001 C CNN
 F 3 "~" H 2050 5950 50  0001 C CNN
 	1    2050 5950
