File: input_buffer_bal_XLR_combo_SMD_1206.kicad_pcb (KiCad board)
At the start: 2 copper layers, 62.5 x 55 mm, 31 parts, among them J1 CH1, J2 CH2, J3 POWER, J4 CH1_OUT, J5 CH2_OUT, U1 LM4562, U2 LM4562

Commit message: minor improvements
Parts:
- C1, C2, C3, C4, C5, C6, C7, C8: footprint Capacitor_SMD:C_1206_3216Metric -> Capacitor_SMD:C_1206_3216Metric_Pad1.42x1.75mm_HandSolder
Other:
- board text added: "Bilous Sound"
- board text added: "Neutrik NCJ6FA-H"

Commit message: minor improvements
Other:
- board text added: "May 2023"
- board text added: "Rev 1.1"
