File: input_buffer_bal_XLR_combo_SMD_1206.kicad_pcb (KiCad board)
At the start: 2 copper layers, 62.5 x 55 mm, 31 parts, among them J1 CH1, J2 CH2, J3 POWER, J4 CH1_OUT, J5 CH2_OUT, U1 LM4562, U2 LM4562

Commit message: minor fixes
Parts:
- moved R10 1.25 mm to (140.5, 131.5)
- moved R5 1.25 mm to (105.0, 131.5)
- moved R6 1.25 mm to (137.5, 131.5)
- moved R7 1.25 mm to (102.0, 131.5)
- moved R8 1.25 mm to (108.0, 131.5)
- moved R9 1.25 mm to (134.5, 131.5)
- moved C5 0.75 mm to (96.8, 122.2)
- moved D1 0.75 mm to (96.8, 128.2)
- moved R1 0.75 mm to (96.8, 125.2)
- moved C7 0.25 mm to (129.2, 122.2)
- moved D3 0.25 mm to (129.2, 128.2)
- moved R3 0.25 mm to (129.2, 125.2)
Routing:
- net GND: track 18.9 -> 9.37 mm, vias 259 -> 279
- net Net-(C5-Pad1): track 11.6 -> 13.8 mm
- net Net-(C8-Pad2): track 12.7 -> 14.6 mm
- net Net-(C7-Pad1): track 12.3 -> 13.8 mm
- net Net-(C6-Pad2): track 12.0 -> 13.2 mm
